File: Controller/PCB/Controller PCB v1.sch (EAGLE design)
At the start: 7 parts, among them IC1 74HC4051N,652, IC2 74HC4051N,652

Commit message: pcb work
Parts:
- added ANALOG_2, ANALOG_3: (no value), pinhead:PINHD-1X10/90
- added IC3, IC4: 74HC4051N,652, 74HC4051N_652:74HC4051N,652
Connections:
- new net Y2_0: ANALOG_2.3, IC3.Y0
- new net Y2_1: ANALOG_2.4, IC3.Y1
- new net Y2_2: ANALOG_2.5, IC3.Y2
- new net Y2_3: ANALOG_2.6, IC3.Y3
- new net Y2_4: ANALOG_2.7, IC3.Y4
- new net Y2_5: ANALOG_2.8, IC3.Y5
- new net Y2_6: ANALOG_2.9, IC3.Y6
- new net Y2_7: ANALOG_2.10, IC3.Y7
- new net Y2_Z: ESP32.IO34, IC3.Z
- new net Y3_0: ANALOG_3.3, IC4.Y0
- new net Y3_1: ANALOG_3.4, IC4.Y1
- new net Y3_2: ANALOG_3.5, IC4.Y2
- new net Y3_3: ANALOG_3.6, IC4.Y3
- new net Y3_4: ANALOG_3.7, IC4.Y4
- new net Y3_5: ANALOG_3.8, IC4.Y5
- new net Y3_6: ANALOG_3.9, IC4.Y6
- new net Y3_7: ANALOG_3.10, IC4.Y7
- new net Y3_Z: ESP32.IO35, IC4.Z
- net +3V3: now also ANALOG_2.2, ANALOG_3.2, IC3.VCC, IC4.VCC
- net GND: now also ANALOG_2.1, ANALOG_3.1, IC3.!E, IC3.GND, IC3.VEE, IC4.!E, IC4.GND, IC4.VEE
- net S_0: now also IC3.S0, IC4.S0
- net S_1: now also IC3.S1, IC4.S1
- net S_2: now also IC3.S2, IC4.S2

Commit message: pcb work, controller code work
Parts:
- added C1: (no value), capacitor-wima:C2.5/2
- added LED: (no value), pinhead:PINHD-2X3
- added R1: 220, rcl:R-US_0204/7
Connections:
- removed net IRQ: NRF24.1
- new net DRONE_LED: ESP32.IO17, LED.3
- new net N$2: LED.2, LED.4, LED.6, R1.2
- new net POWER_LED: ESP32.IO16, LED.5
- new net SOFTWARE_LED: ESP32.IO5, LED.1
- net +3V3: now also C1.2
- net GND: now also C1.1, R1.1
Other:
- note added: "SOFTWARE DRONE POWER"
Changed lines of the file:
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@@
 <part name="+3V11" library="supply1" library_urn="urn:adsk.eagle:library:371" deviceset="+3V3" device=""/>
 <part name="ESP32" library="ESP32-DEVKITV1" deviceset="ESP32DEVKITV1" device=""/>
+<part name="LED" library="pinhead" library_urn="urn:adsk.eagle:library:325" deviceset="PINHD-2X3" device="" package3d_urn="urn:adsk.eagle:package:22462/2"/>
+<part name="R1" library="rcl" library_urn="urn:adsk.eagle:library:334" deviceset="R-US_" device="0204/7" package3d_urn="urn:adsk.eagle:package:23498/2" value="220"/>
+<part name="GND6" library="supply1" library_urn="urn:adsk.eagle:library:371" deviceset="GND" device=""/>
+<part name="C1" library="capacitor-wima" library_urn="urn:adsk.eagle:library:116" deviceset="C" device="2.5/2" package3d_urn="urn:adsk.eagle:package:5415/1"/>
 </parts>
 <sheets>
 <sheet>
 <plain>
+<text x="109.22" y="137.16" size="1.778" layer="91">SOFTWARE
+DRONE
+POWER</text>
 </plain>
 <instances>
@@
 <attribute name="VALUE" x="-24.13" y="127" size="1.778" layer="96"/>
 </instance>
-<instance part="GND4" gate="1" x="-33.02" y="134.62" smashed="yes" rot="R270">
-<attribute name="VALUE" x="-35.56" y="137.16" size="1.778" layer="96" rot="R270"/>
-</instance>
-<instance part="+3V6" gate="G$1" x="-30.48" y="132.08" smashed="yes" rot="R90">
-<attribute name="VALUE" x="-25.4" y="129.54" size="1.778" layer="96" rot="R180"/>
+<instance part="GND4" gate="1" x="-35.56" y="139.7" smashed="yes" rot="R270">
+<attribute name="VALUE" x="-38.1" y="142.24" size="1.778" layer="96" rot="R270"/>
+</instance>
+<instance part="+3V6" gate="G$1" x="-38.1" y="132.08" smashed="yes" rot="R90">
+<attribute name="VALUE" x="-33.02" y="129.54" size="1.778" layer="96" rot="R180"/>
 </instance>
 <instance part="NRF24" gate="A" x="35.56" y="162.56" smashed="yes" rot="R180">
@@
 <instance part="ESP32" gate="G$1" x="35.56" y="127" smashed="yes" rot="R90">
 <attribute name="NAME" x="30.48" y="100.33" size="1.27" layer="95" rot="R180"/>
+</instance>
+<instance part="LED" gate="A" x="93.98" y="139.7" smashed="yes">
+<attribute name="NAME" x="87.63" y="145.415" size="1.778" layer="95"/>
+<attribute name="VALUE" x="87.63" y="132.08" size="1.778" layer="96"/>
+</instance>
+<instance part="R1" gate="G$1" x="106.68" y="129.54" smashed="yes" rot="R90">
+<attribute name="NAME" x="105.1814" y="125.73" size="1.778" layer="95" rot="R90"/>
+<attribute name="VALUE" x="109.982" y="125.73" size="1.778" layer="96" rot="R90"/>
+</instance>
+<instance part="GND6" gate="1" x="106.68" y="121.92" smashed="yes">
+<attribute name="VALUE" x="104.14" y="119.38" size="1.778" layer="96"/>
+</instance>
+<instance part="C1" gate="G$1" x="-33.02" y="137.16" smashed="yes">
+<attribute name="NAME" x="-34.036" y="142.621" size="1.778" layer="95"/>
+<attribute name="VALUE" x="-31.496" y="132.461" size="1.778" layer="96"/>
 </instance>
 </instances>
@@
 </segment>
 <segment>
+<pinref part="GND4" gate="1" pin="GND"/>
+<pinref part="C1" gate="G$1" pin="1"/>
+<wire x1="-33.02" y1="139.7" x2="-27.94" y2="139.7" width="0.1524" layer="91"/>
+<wire x1="-27.94" y1="139.7" x2="-27.94" y2="134.62" width="0.1524" layer="91"/>
+<junction x="-33.02" y="139.7"/>
 <pinref part="BATT" gate="G$1" pin="1"/>
-<pinref part="GND4" gate="1" pin="GND"/>
-<wire x1="-20.32" y1="134.62" x2="-30.48" y2="134.62" width="0.1524" layer="91"/>
+<wire x1="-27.94" y1="134.62" x2="-20.32" y2="134.62" width="0.1524" layer="91"/>
 </segment>
 <segment>
@@
 <pinref part="GND8" gate="1" pin="GND"/>
 </segment>
+<segment>
+<pinref part="GND6" gate="1" pin="GND"/>
+<pinref part="R1" gate="G$1" pin="1"/>
+</segment>
 </net>
 <net name="+3V3" class="0">
@@
 <pinref part="+3V6" gate="G$1" pin="+3V3"/>
 <pinref part="BATT" gate="G$1" pin="2"/>
-<wire x1="-27.94" y1="132.08" x2="-20.32" y2="132.08" width="0.1524" layer="91"/>
+<wire x1="-35.56" y1="132.08" x2="-33.02" y2="132.08" width="0.1524" layer="91"/>
+<pinref part="C1" gate="G$1" pin="2"/>
+<wire x1="-33.02" y1="132.08" x2="-20.32" y2="132.08" width="0.1524" layer="91"/>
+<junction x="-33.02" y="132.08"/>
 </segment>
 <segment>
@@
 </segment>
 </net>
-<net name="IRQ" class="0">
-<segment>
-<pinref part="NRF24" gate="A" pin="1"/>
-<wire x1="38.1" y1="157.48" x2="48.26" y2="157.48" width="0.1524" layer="91"/>
-<label x="43.18" y="157.48" size="1.778" layer="95"/>
-</segment>
-</net>
 <net name="MISO" class="0">
 <segment>
@@
 </segment>
 </net>
+<net name="SOFTWARE_LED" class="0">
+<segment>
+<pinref part="ESP32" gate="G$1" pin="IO5"/>
+<wire x1="53.34" y1="121.92" x2="60.96" y2="121.92" width="0.1524" layer="91"/>
+<wire x1="60.96" y1="121.92" x2="60.96" y2="142.24" width="0.1524" layer="91"/>
+<pinref part="LED" gate="A" pin="1"/>
+<wire x1="91.44" y1="142.24" x2="60.96" y2="142.24" width="0.1524" layer="91"/>
+<label x="66.04" y="142.24" size="1.778" layer="95"/>
+</segment>
+</net>
+<net name="DRONE_LED" class="0">
+<segment>
+<pinref part="ESP32" gate="G$1" pin="IO17"/>
+<wire x1="53.34" y1="119.38" x2="63.5" y2="119.38" width="0.1524" layer="91"/>
+<wire x1="63.5" y1="119.38" x2="63.5" y2="132.08" width="0.1524" layer="91"/>
+<pinref part="LED" gate="A" pin="3"/>
+<wire x1="91.44" y1="139.7" x2="63.5" y2="139.7" width="0.1524" layer="91"/>
+<wire x1="63.5" y1="139.7" x2="63.5" y2="132.08" width="0.1524" layer="91"/>
+<label x="66.04" y="139.7" size="1.778" layer="95"/>
+</segment>
+</net>
+<net name="N$2" class="0">
+<segment>
+<pinref part="LED" gate="A" pin="2"/>
+<wire x1="99.06" y1="142.24" x2="104.14" y2="142.24" width="0.1524" layer="91"/>
+<wire x1="104.14" y1="142.24" x2="104.14" y2="139.7" width="0.1524" layer="91"/>
+<pinref part="LED" gate="A" pin="6"/>
+<wire x1="104.14" y1="139.7" x2="104.14" y2="137.16" width="0.1524" layer="91"/>
+<wire x1="104.14" y1="137.16" x2="99.06" y2="137.16" width="0.1524" layer="91"/>
+<pinref part="LED" gate="A" pin="4"/>
+<wire x1="99.06" y1="139.7" x2="104.14" y2="139.7" width="0.1524" layer="91"/>
+<junction x="104.14" y="139.7"/>
+<wire x1="104.14" y1="139.7" x2="106.68" y2="139.7" width="0.1524" layer="91"/>
+<wire x1="106.68" y1="139.7" x2="106.68" y2="134.62" width="0.1524" layer="91"/>
+<pinref part="R1" gate="G$1" pin="2"/>
+</segment>
+</net>
+<net name="POWER_LED" class="0">
+<segment>
+<pinref part="LED" gate="A" pin="5"/>
+<wire x1="91.44" y1="137.16" x2="66.04" y2="137.16" width="0.1524" layer="91"/>
+<wire x1="66.04" y1="137.16" x2="66.04" y2="116.84" width="0.1524" layer="91"/>
+<pinref part="ESP32" gate="G$1" pin="IO16"/>
+<wire x1="66.04" y1="116.84" x2="53.34" y2="116.84" width="0.1524" layer="91"/>
+<label x="66.04" y="137.16" size="1.778" layer="95"/>
+</segment>
+</net>
 </nets>
 </sheet>
@@
 </drawing>
 <compatibility>
+<note version="6.3" minversion="6.2.2" severity="warning">
+Since Version 6.2.2 text objects can contain more than one line,
+which will not be processed correctly with this version.
+</note>
 <note version="8.2" severity="warning">
 Since Version 8.2, EAGLE supports online libraries. The ids
@@
 packages will not be understood (or retained) with this version.
 </note>
+<note version="8.4" severity="warning">
+Since Version 8.4, EAGLE supports properties for SPICE simulation.
+Probes in schematics and SPICE mapping objects found in parts and library devices
+will not be understood with this version. Update EAGLE to the latest version
+for full support of SPICE simulation.
+</note>
 </compatibility>
